Commit message: UD0117_succeed in controlling_need to adjust the value of pid

File: src/gisbot_localization_1/urdf/inertial_matrix.xacro (robot description, xacro)
@@ -1,4 +1,4 @@
 <?xml version="1.0"?>
-<robot name="base" xmlns:xacro="http://wiki.ros.org/xacro">
+<robot name="my_car" xmlns:xacro="http://wiki.ros.org/xacro">
     <!-- Macro for inertia matrix -->
     <xacro:macro name="sphere_inertial_matrix" params="m r">

File: src/gisbot_localization_1/urdf/my_car_1.urdf.xacro (robot description, xacro)
@@ -6,5 +6,7 @@
     <!--本体-->
     <xacro:include filename="my_car_base_1.xacro" />
+    <xacro:include filename="my_car_gazebo_plugins.xacro" />
     <!--控制器-->
-    <xacro:include filename="my_car_control.urdf.xacro" />
+    <xacro:include filename="my_car_twist.xacro" />
+    <xacro:include filename="my_car_ros_control.xacro" />
 </robot>

File: src/gisbot_localization_1/urdf/my_car_base_1.xacro (robot description, xacro)
@@ -11,5 +11,5 @@
 -->
 <!-- 根标签，必须声明 xmlns:xacro -->
-<robot name="my_base" xmlns:xacro="http://www.ros.org/wiki/xacro">
+<robot name="my_car" xmlns:xacro="http://www.ros.org/wiki/xacro">
     <!-- 封装变量、常量 -->
     <!-- PI 值设置精度需要高一些，否则后续车轮翻转量计算时，可能会出现肉眼不能察觉的车轮倾斜，从而导致模型抖动 -->
@@ -42,7 +42,4 @@
       </visual>
     </link>
-    <gazebo reference="base_footprint">
-      <turnGravityOff>false</turnGravityOff> <!--关闭重力-->
-    </gazebo>
     <!-- 底盘 -->
     <link name="base_link">
@@ -69,7 +66,4 @@
       <origin xyz="0 0 ${earth_space + base_link_z / 2 }" />
     </joint>
-    <gazebo reference="base_link">
-        <material>Gazebo/Yellow</material>
-    </gazebo>
     <!-- 后驱动轮 -->
     <xacro:macro name="add_moving_wheels" params="wheel_name x_flag y_flag">
@@ -96,10 +90,7 @@
         <axis xyz="0 1 0" />
         <dynamics damping="0.0"/>
-		    <limit effort="100" velocity="100"/>
+		    <limit effort="100" velocity="1000"/>
 		    <joint_properties damping="0.0" friction="0.0"/>
       </joint>
-      <gazebo reference="${wheel_name}_wheel">
-        <material>Gazebo/Red</material>
-      </gazebo>
     </xacro:macro>
     <xacro:add_moving_wheels wheel_name="back_left" x_flag="-1" y_flag="1" />
@@ -129,11 +120,11 @@
         <origin xyz="${x_flag * wheel_dis_x *0.5} ${y_flag * wheel_dis_y *0.5} 0.0" />
         <axis xyz="0 0 1" />
-        <dynamics damping="0.0"/>
-        <limit effort="2.5" velocity="10" lower="-0.785" upper="0.785" />
-        <joint_properties damping="20.0" friction="20.0"/>
+        <!--effort最大力/力矩 v速度-->
+        <limit effort="10" velocity="1000" lower="-0.6" upper="0.6" />
+        <!--阻尼系数0-->
+        <dynamics damping="0.1"/>
+        <!--damping阻尼系数 friction摩擦系数-->
+        <joint_properties damping="0.1" friction="1.0"/>
       </joint>
-      <gazebo reference="${joint_name}_wheel_joint">
-        <material>Gazebo/Black</material>
-      </gazebo>
       <!--转向轮-->
       <link name="${joint_name}_wheel">
@@ -159,10 +150,7 @@
         <axis xyz="0 1 0" />
         <dynamics damping="0.0"/>
-        <limit effort="100" velocity="100"/>
-    	<joint_properties damping="0.0" friction="0.0"/>
+        <limit effort="100" velocity="1000"/>
+    	<joint_properties damping="0.0" friction="0.0"/>-->
       </joint>
-      <gazebo reference="${joint_name}_wheel">
-        <material>Gazebo/Red</material>
-      </gazebo>
     </xacro:macro>
     <xacro:add_wheel_joints joint_name="front_left" x_flag="1" y_flag="1" />
